Commit message: Tweaks a bit the compass gait masses

File: underactuated/models/compass_gait.urdf (robot description, URDF)
Before this commit: robot compass_gait, 5 links, 5 joints
Links:
- link ground: geometry collision box size=6 1 .5; visual box size=6 1 .5
- link stance_leg: mass 5 -> .1; geometry collision sphere radius=0; visual cylinder length=1 radius=.01
- link swing_leg: mass 5 -> .1; geometry collision sphere radius=0; visual cylinder length=1 radius=.01

Commit message: Fixes a bug in the compass gait urdf.

File: underactuated/models/compass_gait.urdf (robot description, URDF)
Before this commit: robot compass_gait, 5 links, 5 joints
Links:
- added link body, mass 1; visual sphere radius=.1
- link swing_leg: geometry collision sphere radius=0; visual cylinder length=1 radius=.01
Joints:
- added joint body_on_stance_leg: type fixed, parent stance_leg, child body, origin xyz=0 0 1
- joint hip_pin: origin xyz=0 0 1 -> (none); parent stance_leg -> body

Commit message: Puts the ramp slope in the urdf for the compass gait

File: underactuated/models/compass_gait.urdf (robot description, URDF)
Before this commit: robot compass_gait, 6 links, 6 joints
Joints:
- joint ground_is_world: origin (none) -> xyz=0 0 0 rpy=0 .04 0

Commit message: Removes collisions from the compass gait urdf

File: underactuated/models/compass_gait.urdf (robot description, URDF)
Before this commit: robot compass_gait, 6 links, 6 joints
Links:
- link ground: geometry visual box size=6 1 .5
- link stance_leg: geometry visual cylinder length=1 radius=.01; visual sphere radius=.05
- link swing_leg: geometry visual cylinder length=1 radius=.01; visual sphere radius=.05
