Commit message: Updates the urdf of the compass gait.

File: underactuated/models/compass_gait_abs.urdf (robot description, URDF)
Before this commit: robot compass_gait, 6 links, 6 joints
Links:
- removed link floating_base_z
- link body: mass 1 -> 10
- link stance_leg: mass .1 -> 1
- link swing_leg: mass .1 -> 1
Joints:
- removed joint body_on_stance_leg
- removed joint floating_base_y
- removed joint hip_pin
- added joint stance_hip: type continuous, parent body, child stance_leg, axis 0 -1 0
- added joint swing_hip: type continuous, parent body, child swing_leg, axis 0 -1 0
- joint floating_base_z: child floating_base_z -> body
- joint ground_is_world: origin xyz=0 0 0 rpy=0 .04 0 -> xyz=0 0 0 rpy=0 .0525 0
