Commit message: first pass at perching glider text + code

File: underactuated/models/glider/glider.urdf (robot description, URDF)
Before this commit: robot glider, 8 links, 7 joints
Links:
- removed link fuselageh_hstab
- removed link fuselageh_main
- removed link fuselagev_main
- removed link fuselagev_top
- removed link fuselagev_vstab
- removed link wing_left
- removed link wing_right
- added link fuselage, mass 0.00370301987946561; collision mesh filename=meshes/fuselageh_hstab.obj; collision mesh filename=meshes/fuselageh_main.obj
Joints:
- removed joint fuselageh_hstab
- removed joint fuselageh_main
- removed joint fuselagev_top
- removed joint fuselagev_vstab
- removed joint wing_left
- removed joint wing_right
- joint elevator_hinge: limit lower=-0.8 upper=0.8 effort=0 velocity=0 -> lower=-0.9473 upper=0.4463 effort=0 velocity=0; origin xyz=-0.31696 -0.00014046 0 rpy=0 0 0 -> xyz=-0.317 0 0 rpy=0 0 0; parent fuselagev_main -> fuselage

Commit message: Use URLs for model paths
For packaged models, Drake recommends using URLs (not FindResource).

File: underactuated/models/glider/glider.urdf (robot description, URDF)
Before this commit: robot glider, 2 links, 1 joints
Links:
- link elevator: geometry collision mesh filename=package://underactuated/models/glider/meshes/elevator.obj; visual mesh filename=package://underactuated/models/glider/meshes/elevator.obj
- link fuselage: geometry collision mesh filename=package://underactuated/models/glider/meshes/fuselageh_hsta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; collision mesh filename=package://underactuated/models/glider/meshes/fuselageh_main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
